File: TestKiCadProject/TestKiCadProject.kicad_pcb (KiCad board)
At the start: 2 copper layers, 0 parts

Commit message: Some footprint associations
Parts:
- added C1, C2, C3: 0.1 μ, Capacitors_SMD:C_0603, F.Cu at (148.5, 105.0)
- added J1-UndamnedUSB-IN1: DB15_Male, DSUB:DSUB-15_Male_EdgeMount_Pitch2.77mm, F.Cu at (148.5, 105.0)
- added J2-SNES-OUT1: DB9_Female, DSUB:DSUB-9_Male_EdgeMount_Pitch2.77mm, F.Cu at (148.5, 105.0)
- added J3-NintendoSpy-OUT1: GPIO-3Pin-Female, Pin_Headers:Pin_Header_Angled_1x03_Pitch2.54mm, F.Cu at (148.5, 105.0)
- added R1, R10, R11A1, R11B1, R12, R13, R14, R15, R16, R2, R3, R4, R5, R6, R7, R8, R9: 10k, Resistors_SMD:R_0603, F.Cu at (148.5, 105.0)
- added U1, U2: SN74HC165N, SMD_Packages:SO-16-N, F.Cu at (148.5, 105.0)
- added U3-NAND1: 74HC132N, SMD_Packages:SOIC-14_N, F.Cu at (148.5, 105.0)
Other:
- net class Default: clearance 0.2 -> 0.25
- rule trace_clearance: 0.2 -> 0.25
- rule trace_min: 0.2 -> 0.25
