File: TestKiCadProject/TestKiCadProject.sch (KiCad schematic (older format))
At the start: 26 parts, among them J1-UndamnedUSB-IN1 DB15_Male, J2-SNES-OUT1 DB9_Female, J3-NintendoSpy-OUT1 GPIO-3Pin-Female, U1 SN74HC165N, U2 SN74HC165N, U3-NAND1 74HC132N

Commit message: Some footprint associations
Parts:
- C1, C2, C3: footprint (none) -> Capacitors_SMD:C_0603
- J1-UndamnedUSB-IN1: footprint (none) -> DSUB:DSUB-15_Male_EdgeMount_Pitch2.77mm
- J2-SNES-OUT1: footprint (none) -> DSUB:DSUB-9_Male_EdgeMount_Pitch2.77mm
- J3-NintendoSpy-OUT1: footprint (none) -> Pin_Headers:Pin_Header_Angled_1x03_Pitch2.54mm
- R1, R10, R11A1, R11B1, R12, R13, R14, R15, R16, R2, R3, R4, R5, R6, R7, R8, R9: footprint (none) -> Resistors_SMD:R_0603
- U1, U2: footprint DIP254P762X508-16 -> SMD_Packages:SO-16-N
- U3-NAND1: footprint DIP254P762X420-14 -> SMD_Packages:SOIC-14_N
Changed lines of the file:
@@
 F 0 "R1" V 1550 1650 50  0000 C CNN
 F 1 "10k" V 1550 1900 50  0000 C CNN
-F 2 "" V 1480 1900 50  0001 C CNN
+F 2 "Resistors_SMD:R_0603" V 1480 1900 50  0001 C CNN
 F 3 "" H 1550 1900 50  0001 C CNN
 	1    1550 1900
@@
 F 0 "R2" V 1550 1950 50  0000 C CNN
 F 1 "10k" V 1550 2200 50  0000 C CNN
-F 2 "" V 1480 2200 50  0001 C CNN
+F 2 "Resistors_SMD:R_0603" V 1480 2200 50  0001 C CNN
 F 3 "" H 1550 2200 50  0001 C CNN
 	1    1550 2200
@@
 F 0 "R3" V 1550 1850 50  0000 C CNN
 F 1 "10k" V 1550 2100 50  0000 C CNN
-F 2 "" V 1480 2100 50  0001 C CNN
+F 2 "Resistors_SMD:R_0603" V 1480 2100 50  0001 C CNN
 F 3 "" H 1550 2100 50  0001 C CNN
 	1    1550 2100
@@
 F 0 "R4" V 1550 1750 50  0000 C CNN
 F 1 "10k" V 1550 2000 50  0000 C CNN
-F 2 "" V 1480 2000 50  0001 C CNN
+F 2 "Resistors_SMD:R_0603" V 1480 2000 50  0001 C CNN
 F 3 "" H 1550 2000 50  0001 C CNN
 	1    1550 2000
@@
 F 0 "R5" V 1550 2050 50  0000 C CNN
 F 1 "10k" V 1550 2300 50  0000 C CNN
-F 2 "" V 1480 2300 50  0001 C CNN
+F 2 "Resistors_SMD:R_0603" V 1480 2300 50  0001 C CNN
 F 3 "" H 1550 2300 50  0001 C CNN
 	1    1550 2300
@@
 F 0 "R6" V 1550 2150 50  0000 C CNN
 F 1 "10k" V 1550 2400 50  0000 C CNN
-F 2 "" V 1480 2400 50  0001 C CNN
+F 2 "Resistors_SMD:R_0603" V 1480 2400 50  0001 C CNN
 F 3 "" H 1550 2400 50  0001 C CNN
 	1    1550 2400
@@
 F 0 "R7" V 1550 2250 50  0000 C CNN
 F 1 "10k" V 1550 2500 50  0000 C CNN
-F 2 "" V 1480 2500 50  0001 C CNN
+F 2 "Resistors_SMD:R_0603" V 1480 2500 50  0001 C CNN
 F 3 "" H 1550 2500 50  0001 C CNN
 	1    1550 2500
@@
 F 0 "R8" V 1550 2350 50  0000 C CNN
 F 1 "10k" V 1550 2600 50  0000 C CNN
-F 2 "" V 1480 2600 50  0001 C CNN
+F 2 "Resistors_SMD:R_0603" V 1480 2600 50  0001 C CNN
 F 3 "" H 1550 2600 50  0001 C CNN
 	1    1550 2600
@@
 F 0 "R10" V 4250 2000 50  0000 C CNN
 F 1 "10k" V 4250 2300 50  0000 C CNN
-F 2 "" V 4180 2300 50  0001 C CNN
+F 2 "Resistors_SMD:R_0603" V 4180 2300 50  0001 C CNN
 F 3 "" H 4250 2300 50  0001 C CNN
 	1    4250 2300
@@
 F 0 "R12" V 4250 2200 50  0000 C CNN
 F 1 "10k" V 4250 2500 50  0000 C CNN
-F 2 "" V 4180 2500 50  0001 C CNN
+F 2 "Resistors_SMD:R_0603" V 4180 2500 50  0001 C CNN
 F 3 "" H 4250 2500 50  0001 C CNN
 	1    4250 2500
@@
 F 0 "R13" V 4250 2300 50  0000 C CNN
 F 1 "10k" V 4250 2600 50  0000 C CNN
-F 2 "" V 4180 2600 50  0001 C CNN
+F 2 "Resistors_SMD:R_0603" V 4180 2600 50  0001 C CNN
 F 3 "" H 4250 2600 50  0001 C CNN
 	1    4250 2600
@@
 F 0 "R9" V 4680 1900 50  0000 C CNN
 F 1 "10k" V 4600 1900 50  0000 C CNN
-F 2 "" V 4530 1900 50  0001 C CNN
+F 2 "Resistors_SMD:R_0603" V 4530 1900 50  0001 C CNN
 F 3 "" H 4600 1900 50  0001 C CNN
 	1    4600 1900
@@
 F 0 "J1-UndamnedUSB-IN1" H 8650 2700 50  0000 C CNN
 F 1 "DB15_Male" H 8200 975 50  0000 C CNN
-F 2 "" H 8200 1850 50  0001 C CNN
+F 2 "DSUB:DSUB-15_Male_EdgeMount_Pitch2.77mm" H 8200 1850 50  0001 C CNN
 F 3 "" H 8200 1850 50  0001 C CNN
 	1    8200 1850
@@
 F 0 "U2" H 5493 2879 50  0000 L BNN
 F 1 "SN74HC165N" H 5500 700 50  0000 L BNN
-F 2 "DIP254P762X508-16" H 5700 1900 50  0001 L BNN
+F 2 "SMD_Packages:SO-16-N" H 5700 1900 50  0001 L BNN
 F 3 "None" H 5700 1900 50  0001 L BNN
 F 4 "PDIP-16 STMicroelectronics" H 5700 1900 50  0001 L BNN "Field4"
@@
 F 0 "R11B1" V 1850 4150 50  0000 C CNN
 F 1 "10k" V 1800 4400 50  0000 C CNN
-F 2 "" V 1730 4400 50  0001 C CNN
+F 2 "Resistors_SMD:R_0603" V 1730 4400 50  0001 C CNN
 F 3 "" H 1800 4400 50  0001 C CNN
 	1    1800 4400
@@
 F 0 "J2-SNES-OUT1" H 8450 4550 50  0000 C CNN
 F 1 "DB9_Female" H 8200 3425 50  0000 C CNN
-F 2 "" H 8200 4000 50  0001 C CNN
+F 2 "DSUB:DSUB-9_Male_EdgeMount_Pitch2.77mm" H 8200 4000 50  0001 C CNN
 F 3 "" H 8200 4000 50  0001 C CNN
 	1    8200 4000
@@
 F 0 "R14" V 5480 4800 50  0000 C CNN
 F 1 "10k" V 5400 4800 50  0000 C CNN
-F 2 "" V 5330 4800 50  0001 C CNN
+F 2 "Resistors_SMD:R_0603" V 5330 4800 50  0001 C CNN
 F 3 "" H 5400 4800 50  0001 C CNN
 	1    5400 4800
@@
 F 0 "R15" V 5480 4950 50  0000 C CNN
 F 1 "10k" V 5400 4950 50  0000 C CNN
-F 2 "" V 5330 4950 50  0001 C CNN
+F 2 "Resistors_SMD:R_0603" V 5330 4950 50  0001 C CNN
 F 3 "" H 5400 4950 50  0001 C CNN
 	1    5400 4950
@@
 F 0 "R16" V 5480 5100 50  0000 C CNN
 F 1 "10k" V 5400 5100 50  0000 C CNN
-F 2 "" V 5330 5100 50  0001 C CNN
+F 2 "Resistors_SMD:R_0603" V 5330 5100 50  0001 C CNN
 F 3 "" H 5400 5100 50  0001 C CNN
 	1    5400 5100
@@
 F 0 "J3-NintendoSpy-OUT1" H 6050 5200 50  0000 C CNN
 F 1 "GPIO-3Pin-Female" H 6000 4750 50  0000 C CNN
-F 2 "" H 6200 4950 50  0001 C CNN
+F 2 "Pin_Headers:Pin_Header_Angled_1x03_Pitch2.54mm" H 6200 4950 50  0001 C CNN
 F 3 "" H 6200 4950 50  0001 C CNN
 	1    6200 4950
@@
 F 0 "C1" V 4850 1050 50  0000 L CNN
 F 1 "0.1 μ" V 4750 1050 50  0000 L CNN
-F 2 "" H 4900 1200 50  0001 C CNN
+F 2 "Capacitors_SMD:C_0603" H 4900 1200 50  0001 C CNN
 F 3 "" H 4900 1200 50  0001 C CNN
 	1    4900 1200
@@
 F 0 "C2" V 1950 1050 50  0000 L CNN
 F 1 "0.1 μ" V 1850 1050 50  0000 L CNN
-F 2 "" H 2000 1200 50  0001 C CNN
+F 2 "Capacitors_SMD:C_0603" H 2000 1200 50  0001 C CNN
 F 3 "" H 2000 1200 50  0001 C CNN
 	1    2000 1200
@@
 F 0 "C3" V 1900 3550 50  0000 L CNN
 F 1 "0.1 μ" V 1800 3500 50  0000 L CNN
-F 2 "" H 1950 3700 50  0001 C CNN
+F 2 "Capacitors_SMD:C_0603" H 1950 3700 50  0001 C CNN
 F 3 "" H 1950 3700 50  0001 C CNN
 	1    1950 3700
@@
 F 0 "R11A1" V 1850 3650 50  0000 C CNN
 F 1 "10k" V 1800 3900 50  0000 C CNN
-F 2 "" V 1730 3900 50  0001 C CNN
+F 2 "Resistors_SMD:R_0603" V 1730 3900 50  0001 C CNN
 F 3 "" H 1800 3900 50  0001 C CNN
 	1    1800 3900
@@
 F 0 "U1" H 2593 2879 50  0000 L BNN
 F 1 "SN74HC165N" H 2600 700 50  0000 L BNN
-F 2 "DIP254P762X508-16" H 2800 1900 50  0001 L BNN
+F 2 "SMD_Packages:SO-16-N" H 2800 1900 50  0001 L BNN
 F 3 "None" H 2800 1900 50  0001 L BNN
 F 4 "PDIP-16 STMicroelectronics" H 2800 1900 50  0001 L BNN "Field4"
@@
 F 0 "U3-NAND1" H 2550 5100 50  0000 L BNN
 F 1 "74HC132N" H 2600 3350 50  0000 L BNN
-F 2 "DIP254P762X420-14" H 2750 4350 50  0001 L BNN
+F 2 "SMD_Packages:SOIC-14_N" H 2750 4350 50  0001 L BNN
 F 3 "NAND Gate 4-Element 2-IN CMOS 14-Pin PDIP Bulk" H 2750 4350 50  0001 L BNN
 F 4 "Unavailable" H 2750 4350 50  0001 L BNN "Field4"
